Commit message: descripción del moveit y del robot

File: urdf/urdf.xacro (robot description, xacro)
@@ -1,27 +1,44 @@
 <?xml version="1.0"?>
-<robot xmlns:xacro="http://www.ros.org/wiki/xacro" name="peacetolero/">
-  <!-- Parameters -->
-  <xacro:property name="prefix" value=""/>
-  <!-- Base Link -->
-  <link name="${prefix}base_link">
-    <visual>
-      <geometry>
-        <mesh filename="package://peacetolero_description/meshes/peacetolero.dae" scale="1 1 1"/>
-      </geometry>
-      <material name="blue">
-        <color rgba="0 0 1 1"/>
-      </material>
-    </visual>
-    <collision>
-      <geometry>
-        <mesh filename="package://peacetolero_description/meshes/peacetolero.dae" scale="1 1 1"/>
-      </geometry>
-    </collision>
-    <inertial>
-      <mass value="1.0"/>
-      <origin xyz="0 0 0" rpy="0 0 0"/>
-      <inertia ixx="0.1" ixy="0.0" ixz="0.0"
-              iyy="0.1" iyz="0.0" izz="0.1"/>
-    </inertial>
-  </link>
+<robot xmlns:xacro="http://www.ros.org/wiki/xacro" name="peacetolero">
+  <!-- Definir un macro llamado peacetolero_macro -->
+  <xacro:macro name="peacetolero_macro" params="prefix">
+    <!-- Base Link -->
+    <link name="${prefix}base_link">
+      <visual>
+        <origin rpy="0 0 1.5708" xyz="0 0 0" />
+        <geometry>
+          <mesh filename="package://peacetolero_description/meshes/peacetolero.dae" scale="1 1 1"/>
+        </geometry>
+        <material name="blue">
+          <color rgba="0 0 1 1"/>
+        </material>
+      </visual>
+      <collision>
+        <geometry>
+          <mesh filename="package://peacetolero_description/meshes/peacetolero.dae" scale="1 1 1"/>
+        </geometry>
+      </collision>
+    </link>
+    <link name="${prefix}alpha_suport">
+      <visual>
+        <origin rpy="0 0 1.5708" xyz="0 0 0" />
+        <geometry>
+          <mesh filename="package://peacetolero_description/meshes/soporte_alpha.dae" scale="1 1 1"/>
+        </geometry>
+        <material name="blue">
+          <color rgba="0 0 1 1"/>
+        </material>
+      </visual>
+      <collision>
+        <geometry>
+          <mesh filename="package://peacetolero_description/meshes/soporte_alpha.dae" scale="1 1 1"/>
+        </geometry>
+      </collision>
+    </link>
+    <joint name="base_link2arm" type="fixed">
+      <parent link="${prefix}base_link"/>
+      <child link="${prefix}alpha_suport"/>
+      <origin xyz="0.0 0.0 0.0" rpy="0 0 0" />
+    </joint>
+  </xacro:macro>
 </robot>

Commit message: Ajuste de planning con moveit para peacetolero

File: urdf/urdf.xacro (robot description, xacro)
@@ -15,4 +15,5 @@
       </visual>
       <collision>
+        <origin rpy="0 0 1.5708" xyz="0 0 0" />
         <geometry>
           <mesh filename="package://peacetolero_description/meshes/peacetolero.dae" scale="1 1 1"/>

Commit message: ajuste en la posicion del brazo y escena de moveit con el pipe

File: urdf/urdf.xacro (robot description, xacro)
@@ -23,5 +23,5 @@
     <link name="${prefix}alpha_suport">
       <visual>
-        <origin rpy="0 0 1.5708" xyz="0 0 0" />
+        <origin rpy="0 0 1.5708" xyz="0 0.11 0" />
         <geometry>
           <mesh filename="package://peacetolero_description/meshes/soporte_alpha.dae" scale="1 1 1"/>
@@ -32,4 +32,5 @@
       </visual>
       <collision>
+        <origin rpy="0 0 1.5708" xyz="0 0.11 0" />
         <geometry>
           <mesh filename="package://peacetolero_description/meshes/soporte_alpha.dae" scale="1 1 1"/>

Commit message: Ajuste de soporte alpha para posición real

File: urdf/urdf.xacro (robot description, xacro)
@@ -23,5 +23,5 @@
     <link name="${prefix}alpha_suport">
       <visual>
-        <origin rpy="0 0 1.5708" xyz="0 0.11 0" />
+        <origin rpy="0 0 1.5708" xyz="0 0 0" />
         <geometry>
           <mesh filename="package://peacetolero_description/meshes/soporte_alpha.dae" scale="1 1 1"/>
@@ -32,5 +32,5 @@
       </visual>
       <collision>
-        <origin rpy="0 0 1.5708" xyz="0 0.11 0" />
+        <origin rpy="0 0 1.5708" xyz="0 0 0" />
         <geometry>
           <mesh filename="package://peacetolero_description/meshes/soporte_alpha.dae" scale="1 1 1"/>
