Commit message: actualizacion de ruedas

File: urdf/peacetolero_alpha.config.xacro (robot description, xacro)
@@ -8,5 +8,6 @@
   <xacro:arg name="initial_positions_file" default="initial_positions.yaml" />
   <xacro:arg name="namespace" default="" />
-  <xacro:arg name="prefix" default="peacetolero_" />
+  <!-- cambie el _ por / en  default="peacetolero_" -->
+  <xacro:arg name="prefix" default="peacetolero/" />
   <xacro:arg name="use_sim" default="false" />
   <xacro:arg name="alpha_description_package" default="alpha_description" />
@@ -21,5 +22,6 @@
   <xacro:peacetolero_alpha prefix="$(arg prefix)">
   </xacro:peacetolero_alpha>
-  <xacro:alpha_system prefix="$(arg prefix)alpha_" name="ReachAlpha5" serial_port="$(arg serial_port)"
+  <!-- cambie el _ por / en  prefix="$(arg prefix)alpha_" -->
+  <xacro:alpha_system prefix="$(arg prefix)_alpha/" name="ReachAlpha5" serial_port="$(arg serial_port)"
     state_update_frequency="$(arg state_update_frequency)"
     initial_positions_file="$(arg initial_positions_file)"

File: urdf/peacetolero_alpha.xacro (robot description, xacro)
@@ -12,5 +12,6 @@
     <xacro:peacetolero_macro prefix="$(arg prefix)" />
     <!-- Instanciar el alpha.urdf.xacro -->
-    <xacro:alpha_urdf parent="$(arg prefix)base_link" prefix="$(arg prefix)alpha_"
+    <!-- cambie el _ por / en  prefix="$(arg prefix)alpha_" -->
+    <xacro:alpha_urdf parent="$(arg prefix)base_link" prefix="$(arg prefix)alpha/"
       description_package="${description_package}">
       <origin xyz="0.404 0.03 -0.048" rpy="0 0 0" />

File: urdf/urdf.xacro (robot description, xacro)
@@ -6,7 +6,9 @@
     <link name="${prefix}base_link">
       <visual>
-        <origin rpy="0 0 1.5708" xyz="0 0 0" />
+        <!-- <origin rpy="0 0 1.5708" xyz="0 0 0" /> -->
+        <origin rpy="0 1.5708 0" xyz="0 0 0" />
         <geometry>
-          <mesh filename="package://peacetolero_description/meshes/peacetolero.dae" scale="1 1 1"/>
+          <!-- <mesh filename="package://peacetolero_description/meshes/peacetolero.dae" scale="1 1 1"/> -->
+          <mesh filename="package://peacetolero_description/meshes/peacetolero_wheels.dae" scale="1 1 1"/>
         </geometry>
         <material name="blue">
@@ -15,7 +17,8 @@
       </visual>
       <collision>
-        <origin rpy="0 0 1.5708" xyz="0 0 0" />
+        <!-- <origin rpy="0 0 1.5708" xyz="0 0 0" /> -->
+        <origin rpy="0 1.5708 0.0" xyz="0 0 0" />
         <geometry>
-          <mesh filename="package://peacetolero_description/meshes/peacetolero.dae" scale="1 1 1"/>
+          <mesh filename="package://peacetolero_description/meshes/peacetolero_wheels.dae" scale="1 1 1"/>
         </geometry>
       </collision>

Commit message: Ajuste de nombre de joints a peacetolero/alpha_axis***

File: urdf/peacetolero_alpha.config.xacro (robot description, xacro)
@@ -10,5 +10,6 @@
   <!-- cambie el _ por / en  default="peacetolero_" -->
   <xacro:arg name="prefix" default="peacetolero/" />
-  <xacro:arg name="use_sim" default="false" />
+  <!-- importante para stonefish -->
+  <xacro:arg name="use_sim" default="true" />
   <xacro:arg name="alpha_description_package" default="alpha_description" />
   <xacro:arg name="robot_description_package" default="peacetolero_description" />
@@ -23,5 +24,5 @@
   </xacro:peacetolero_alpha>
   <!-- cambie el _ por / en  prefix="$(arg prefix)alpha_" -->
-  <xacro:alpha_system prefix="$(arg prefix)_alpha/" name="ReachAlpha5" serial_port="$(arg serial_port)"
+  <xacro:alpha_system prefix="$(arg prefix)alpha_" name="ReachAlpha5" serial_port="$(arg serial_port)"
     state_update_frequency="$(arg state_update_frequency)"
     initial_positions_file="$(arg initial_positions_file)"

File: urdf/peacetolero_alpha.xacro (robot description, xacro)
@@ -13,5 +13,5 @@
     <!-- Instanciar el alpha.urdf.xacro -->
     <!-- cambie el _ por / en  prefix="$(arg prefix)alpha_" -->
-    <xacro:alpha_urdf parent="$(arg prefix)base_link" prefix="$(arg prefix)alpha/"
+    <xacro:alpha_urdf parent="$(arg prefix)base_link" prefix="$(arg prefix)alpha_"
       description_package="${description_package}">
       <origin xyz="0.404 0.03 -0.048" rpy="0 0 0" />

File: urdf/urdf.xacro (robot description, xacro)
@@ -6,6 +6,6 @@
     <link name="${prefix}base_link">
       <visual>
-        <!-- <origin rpy="0 0 1.5708" xyz="0 0 0" /> -->
-        <origin rpy="0 1.5708 0" xyz="0 0 0" />
+        <origin rpy="0 0 1.5708" xyz="0 0 0" />
+        <!-- <origin rpy="0 1.5708 0" xyz="0 0 0" /> -->
         <geometry>
           <!-- <mesh filename="package://peacetolero_description/meshes/peacetolero.dae" scale="1 1 1"/> -->
