Commit message: ajuste de urdf del peacetolero

File: urdf/peacetolero_alpha.xacro (robot description, xacro)
@@ -14,5 +14,5 @@
     <xacro:alpha_urdf parent="$(arg prefix)base_link" prefix="$(arg prefix)alpha_"
       description_package="${description_package}">
-      <origin xyz="0.404 -0.022 -0.048" rpy="0 0 0" />
+      <origin xyz="0.404 0.03 -0.048" rpy="0 0 0" />
     </xacro:alpha_urdf>
   </xacro:macro>

Commit message: Ajuste orientacion para trabajar con ned y stonefish

File: urdf/peacetolero_alpha.xacro (robot description, xacro)
@@ -15,5 +15,5 @@
     <xacro:alpha_urdf parent="$(arg prefix)base_link" prefix="$(arg prefix)alpha_"
       description_package="${description_package}">
-      <origin xyz="0.404 0.03 -0.048" rpy="0 0 0" />
+      <origin xyz="0.404 -0.03 0.048" rpy="3.1416 0 0" />
     </xacro:alpha_urdf>
   </xacro:macro>

File: urdf/urdf.xacro (robot description, xacro)
@@ -6,5 +6,5 @@
     <link name="${prefix}base_link">
       <visual>
-        <origin rpy="0 0 1.5708" xyz="0 0 0" />
+        <origin rpy="3.1416 0 -1.5708" xyz="0 0 0" />
         <!-- <origin rpy="0 1.5708 0" xyz="0 0 0" /> -->
         <geometry>
@@ -18,5 +18,5 @@
       <collision>
         <!-- <origin rpy="0 0 1.5708" xyz="0 0 0" /> -->
-        <origin rpy="0 1.5708 0.0" xyz="0 0 0" />
+        <origin rpy="3.1416 0.0 -1.5708" xyz="0 0 0" />
         <geometry>
           <mesh filename="package://peacetolero_description/meshes/peacetolero_wheels.dae" scale="1 1 1"/>
@@ -44,5 +44,21 @@
       <parent link="${prefix}base_link"/>
       <child link="${prefix}alpha_suport"/>
-      <origin xyz="0.0 0.0 0.0" rpy="0 0 0" />
+      <origin xyz="0.0 0.0 0.0" rpy="3.1416 0 0" />
+    </joint>
+    <link name="${prefix}zed_camera_link">
+    </link>
+    <link name="${prefix}zed_camera_link1">
+    </link>
+    <!-- Define the fixed joint between base_link and zed_camera_link -->
+    <joint name="base_to_zed" type="fixed">
+      <parent link="${prefix}base_link"/>
+      <child link="${prefix}zed_camera_link"/>
+      <origin xyz="0.2 0.0 0.0" rpy="1.57 3.1416 1.57"/>  <!-- Position and orientation of ZED relative to base_link -->
+    </joint>
+    <!-- Define the fixed joint between base_link and zed_camera_link -->
+    <joint name="base_to_zed1" type="fixed">
+      <parent link="${prefix}base_link"/>
+      <child link="${prefix}zed_camera_link1"/>
+      <origin xyz="0.2 0.0 0.0" rpy="1.57 3.1416 1.57"/>  <!-- Position and orientation of ZED relative to base_link -->
     </joint>
   </xacro:macro>
